File: HelpDuinoShiled.brd (EAGLE design)
At the start: 68 x 59.7 mm, 17 parts, among them IC1 REG1117

Commit message: Finalizing V2 and Ordering
Parts:
- removed LSP1: SE13, solpad:SE13
- added U$2: (no value), digital-ic:FACELOGO
- moved LSP2 4.43 mm to (6.25, 31.4)
- moved LSP3 4.31 mm to (3.05, 29.7)
- moved LSP13 3.90 mm to (6.25, 27.7)
- moved LSP4 2.96 mm to (9.75, 27.7)
- moved C3 0.22 mm to (17.1, 25.1)
Connections:
- removed net 3.3V: C1.1, C3.1, IC1.2
- net 3V3: now also C1.1, C3.1, IC1.2
Routing:
- net 3V3: track 2.59 -> 39.5 mm, vias 0 -> 1
- net N$2: track 32.3 -> 0.00 mm
- net 5V: track 99.9 -> 117.0 mm, vias 6 -> 4
- net 3.3V: track 9.51 -> 0.00 mm
- net D3: track 129.0 -> 125.3 mm
- net N$1: track 1.07 -> 0.00 mm
- net D0: track 72.5 -> 73.2 mm
- net A3: track 33.9 -> 34.6 mm
- net D2: track 118.6 -> 119.0 mm, vias 1 -> 5
- net D8: track 86.3 -> 86.4 mm, vias 5 -> 7
- net RST: vias 2 -> 4
- net A5: vias 4 -> 3
- removed copper zone on layer 16, net 5V
Other:
- board text added: "By:"

Commit message: Adding screenshots
Other:
- board text removed: "56mm entre conector chico y grande Entre parte de afuera Cada pieza mide 5mm de ancho Centro a centro = 46mm 56mm -10mm = 46mm 19mm desde parte de arriba dual pin is @ 22mm from border Short ISP is @ 9mm from border Short ISP header is 8mm long Long double is 31mm len 22-9-4 = 9 9+15.5 = 32.5"
Changed lines of the file:
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@@
 <wire x1="65.55985" y1="58.643" x2="65.27946875" y2="58.921540625" width="0" layer="20"/>
 <wire x1="65.27946875" y1="58.921540625" x2="63.43983125" y2="59.68" width="0" layer="20" curve="44.811368"/>
-<text x="73.47" y="33.21" size="1.778" layer="48">56mm entre conector chico y grande
-Entre parte de afuera
-Cada pieza mide 5mm de ancho
-Centro a centro = 46mm
-56mm -10mm = 46mm
-19mm desde parte de arriba
-dual pin is @ 22mm from border
-Short ISP is @ 9mm from border
-Short ISP header is 8mm long
-Long double is 31mm len
-22-9-4 = 9
-9+15.5 = 32.5</text>
 <text x="3.9624" y="32.9184" size="1.778" layer="21" rot="R90">By:</text>
 <text x="64.008" y="48.768" size="1.016" layer="25" rot="R90">D0\\RX</text>
@@
 </board>
 </drawing>
-<compatibility>
-<note version="6.3" minversion="6.2.2" severity="warning">
-Since Version 6.2.2 text objects can contain more than one line,
-which will not be processed correctly with this version.
-</note>
-</compatibility>
 </eagle>
