File: HelpDuinoShiled.sch (EAGLE design)
At the start: 16 parts, among them IC1 REG1117

Commit message: Finalizing V2 and Ordering
Parts:
- removed LSP1: SE13, solpad:SE13
Connections:
- removed net 3.3V: C1.1, C3.1, IC1.VOUT
- net 3V3: now also C1.1, C3.1, IC1.VOUT

Commit message: Adding screenshots
Other:
- note added: "Power Regulator"
- note added: "Shield pinout"
- moved on the sheet: JP1
